File: Proyecto KICAD/ESP32/ESP32.kicad_pcb (KiCad board)
At the start: 2 copper layers, 34 parts, among them J1 Conn_01x17, J2 Conn_01x17, J3 USB_B_Micro, Q1 BC847, Q2 BC847, SW1 SW_Push, SW2 SW_Push, U1 esp32-devkitM-1, U2 CP2102N-Axx-xQFN28, U3 SGM2212-3.3XKC3G/TR

Commit message: b
Parts:
- moved J2 83.4 mm to (187.9, 86.8)
- moved C7 73.3 mm to (173.6, 117.2), turned to 180 degrees
- moved C8 72.5 mm to (173.6, 119.3), turned to 180 degrees
- moved J3 69.6 mm to (175.1, 124.3)
- moved R3 68.7 mm to (177.3, 111.0)
- moved R8 67.3 mm to (179.9, 114.4), turned to -90 degrees
- moved R7 66.9 mm to (180.5, 107.3)
- moved R2 66.9 mm to (173.8, 110.9)
- moved R4 65.2 mm to (173.8, 113.2)
- moved C10 63.4 mm to (170.7, 116.3), turned to -90 degrees
- moved C11 63.0 mm to (170.1, 119.3)
- moved Q2 62.7 mm to (180.8, 104.4)
- moved J1 61.9 mm to (159.5, 86.8)
- moved U3 61.3 mm to (177.2, 116.2), turned to -90 degrees
- moved C6 60.7 mm to (182.9, 100.5), turned to -90 degrees
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
Commit message: c
Parts:
- U1: footprint nuevas huella:esp32-devkitM-1 -> ESP32-MINI-1U-N4 (3):MODULE_ESP32-MINI-1U-N4
- U3: footprint Package_TO_SOT_SMD:SOT-23 -> Package_TO_SOT_SMD:SOT-223-3_TabPin2
- moved C9 34.4 mm to (182.6, 131.2), turned to 90 degrees
- moved SW2 34.4 mm to (186.6, 131.2), turned to 180 degrees
- moved SW1 33.3 mm to (165.6, 130.9), turned to 180 degrees
- moved C6 33.0 mm to (169.9, 130.8), turned to 90 degrees
- moved Q1 25.9 mm to (184.5, 121.7), turned to -90 degrees
- moved R1 23.6 mm to (183.1, 102.6)
- moved C3 22.7 mm to (185.3, 102.6), turned to 90 degrees
- moved R6 22.1 mm to (185.3, 117.6), turned to -90 degrees
- moved C2 17.8 mm to (166.7, 106.9), turned to -90 degrees
- moved C1 15.0 mm to (168.1, 101.8)
- moved D2 13.9 mm to (167.2, 119.2), turned to 180 degrees
- moved C11 13.6 mm to (164.4, 106.9), turned to -90 degrees
- moved C8 13.2 mm to (168.8, 106.9), turned to -90 degrees
- moved C10 12.6 mm to (168.1, 104.0), turned to 180 degrees
- moved U3 12.0 mm to (175.3, 104.4), turned to 0 degrees
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Connections:
- C10 pad 1: +3V3 -> +3.3V
- C11 pad 1: +3V3 -> +3.3V
- R8 pad 2: +3V3 -> +3.3V
- U1 pad 3: unconnected-(U1-3V3-Pad3) -> +3.3V
- U3 pad 2: +3V3 -> +3.3V
Routing:
- net ESP_RST: track 0.00 -> 111.2 mm, vias 0 -> 6
- net GND: track 0.00 -> 108.4 mm, vias 0 -> 32
- net GPIO12: track 0.00 -> 68.3 mm, vias 0 -> 1
- net GPIO0: track 0.00 -> 66.0 mm, vias 0 -> 2
- net U0RXD: track 0.00 -> 56.0 mm, vias 0 -> 2
- net GPIO13: track 0.00 -> 44.6 mm
- net GPIO14: track 0.00 -> 41.3 mm
- net U0TXD: track 0.00 -> 40.9 mm, vias 0 -> 1
- net GPIO15: track 0.00 -> 40.0 mm
- net +5V: track 0.00 -> 38.7 mm, vias 0 -> 5
- net GPIO2: track 0.00 -> 36.3 mm
- net GPIO27: track 0.00 -> 35.4 mm
- net GPIO26: track 0.00 -> 34.3 mm
- net USB_DP: track 0.00 -> 32.1 mm
- net GPIO4: track 0.00 -> 31.2 mm
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- added copper zone on In2.Cu, net +3.3V
- added copper zone on In1.Cu, net GND
Other:
- board outline added: 44.4 x 58.4 mm
- copper layers 2 -> 4

Commit message: l
Parts:
- added REF**: MountingHole_2.2mm_M2_Pad, MountingHole:MountingHole_2.2mm_M2_Pad, F.Cu at (157.1, 135.4)
- added REF**: MountingHole_2.2mm_M2_Pad, MountingHole:MountingHole_2.2mm_M2_Pad, F.Cu at (157.6, 84.2)
- added REF**: MountingHole_2.2mm_M2_Pad, MountingHole:MountingHole_2.2mm_M2_Pad, F.Cu at (195.5, 84.6)
- added REF**: MountingHole_2.2mm_M2_Pad, MountingHole:MountingHole_2.2mm_M2_Pad, F.Cu at (196.1, 135.5)
Changed lines of the file:
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@@
     )
+  )
+  (footprint "MountingHole:MountingHole_2.2mm_M2_Pad" (layer "F.Cu")
+    (at 157.099 135.382)
+    (descr "Mounting Hole 2.2mm, M2")
+    (tags "mounting hole 2.2mm m2")
+    (attr exclude_from_pos_files exclude_from_bom)
+    (fp_text reference "REF**" (at 0 -3.2) (layer "F.SilkS")
+        (effects (font (size 1 1) (thickness 0.15)))
+    )
+    (fp_text value "MountingHole_2.2mm_M2_Pad" (at 0 3.2) (layer "F.Fab")
+        (effects (font (size 1 1) (thickness 0.15)))
+    )
+    (fp_text user "${REFERENCE}" (at 0 0) (layer "F.Fab")
+        (effects (font (size 1 1) (thickness 0.15)))
+    )
+    (fp_circle (center 0 0) (end 2.2 0)
+      (stroke (width 0.15) (type solid)) (fill none) (layer "Cmts.User"))
+    (fp_circle (center 0 0) (end 2.45 0)
+      (stroke (width 0.05) (type solid)) (fill none) (layer "F.CrtYd"))
+    (pad "1" thru_hole circle (at 0 0) (size 4.4 4.4) (drill 2.2) (layers "*.Cu" "*.Mask"))
   )
   (footprint "Connector_PinHeader_2.54mm:PinHeader_1x17_P2.54mm_Vertical" (layer "F.Cu")
@@
     )
   )
+  (footprint "MountingHole:MountingHole_2.2mm_M2_Pad" (layer "F.Cu")
+    (at 157.607 84.201)
+    (descr "Mounting Hole 2.2mm, M2")
+    (tags "mounting hole 2.2mm m2")
+    (attr exclude_from_pos_files exclude_from_bom)
+    (fp_text reference "REF**" (at 0 -3.2) (layer "F.SilkS")
+        (effects (font (size 1 1) (thickness 0.15)))
+    )
+    (fp_text value "MountingHole_2.2mm_M2_Pad" (at 0 3.2) (layer "F.Fab")
+        (effects (font (size 1 1) (thickness 0.15)))
+    )
+    (fp_text user "${REFERENCE}" (at 0 0) (layer "F.Fab")
+        (effects (font (size 1 1) (thickness 0.15)))
+    )
+    (fp_circle (center 0 0) (end 2.2 0)
+      (stroke (width 0.15) (type solid)) (fill none) (layer "Cmts.User"))
+    (fp_circle (center 0 0) (end 2.45 0)
+      (stroke (width 0.05) (type solid)) (fill none) (layer "F.CrtYd"))
+    (pad "1" thru_hole circle (at 0 0) (size 4.4 4.4) (drill 2.2) (layers "*.Cu" "*.Mask"))
+  )
   (footprint "Capacitor_SMD:C_0805_2012Metric" (layer "F.Cu")
     (at 168.0972 109.7788 180)
@@
       (net 2 "GND") (pinfunction "GND") (pintype "output"))
   )
+  (footprint "MountingHole:MountingHole_2.2mm_M2_Pad" (layer "F.Cu")
+    (at 195.453 84.582)
+    (descr "Mounting Hole 2.2mm, M2")
+    (tags "mounting hole 2.2mm m2")
+    (attr exclude_from_pos_files exclude_from_bom)
+    (fp_text reference "REF**" (at 0 -3.2) (layer "F.SilkS")
+        (effects (font (size 1 1) (thickness 0.15)))
+    )
+    (fp_text value "MountingHole_2.2mm_M2_Pad" (at 0 3.2) (layer "F.Fab")
+        (effects (font (size 1 1) (thickness 0.15)))
+    )
+    (fp_text user "${REFERENCE}" (at 0 0) (layer "F.Fab")
+        (effects (font (size 1 1) (thickness 0.15)))
+    )
+    (fp_circle (center 0 0) (end 2.2 0)
+      (stroke (width 0.15) (type solid)) (fill none) (layer "Cmts.User"))
+    (fp_circle (center 0 0) (end 2.45 0)
+      (stroke (width 0.05) (type solid)) (fill none) (layer "F.CrtYd"))
+    (pad "1" thru_hole circle (at 0 0) (size 4.4 4.4) (drill 2.2) (layers "*.Cu" "*.Mask"))
+  )
+  (footprint "MountingHole:MountingHole_2.2mm_M2_Pad" (layer "F.Cu")
+    (at 196.088 135.509)
+    (descr "Mounting Hole 2.2mm, M2")
+    (tags "mounting hole 2.2mm m2")
+    (attr exclude_from_pos_files exclude_from_bom)
+    (fp_text reference "REF**" (at 0 -3.2) (layer "F.SilkS")
+        (effects (font (size 1 1) (thickness 0.15)))
+    )
+    (fp_text value "MountingHole_2.2mm_M2_Pad" (at 0 3.2) (layer "F.Fab")
+        (effects (font (size 1 1) (thickness 0.15)))
+    )
+    (fp_text user "${REFERENCE}" (at 0 0) (layer "F.Fab")
+        (effects (font (size 1 1) (thickness 0.15)))
+    )
+    (fp_circle (center 0 0) (end 2.2 0)
+      (stroke (width 0.15) (type solid)) (fill none) (layer "Cmts.User"))
+    (fp_circle (center 0 0) (end 2.45 0)
+      (stroke (width 0.05) (type solid)) (fill none) (layer "F.CrtYd"))
+    (pad "1" thru_hole circle (at 0 0) (size 4.4 4.4) (drill 2.2) (layers "*.Cu" "*.Mask"))
+  )
   (footprint "LED_SMD:LED_0805_2012Metric" (layer "F.Cu")
