File: Proyecto KICAD/RoomLink/RS-485-EXTERNA.kicad_sch (KiCad schematic)
At the start: 11 parts, among them U8 TD521D485H-E

Commit message: PCB
Connections:
- net +5V renamed VDD
Changed lines of the file:
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@@
     (stroke (width 0) (type default))
   )
-  (wire (pts (xy 96.52 98.044) (xy 100.33 98.044))
+  (wire (pts (xy 96.52 98.044) (xy 104.648 98.044))
     (stroke (width 0) (type default))
   )
@@
   )
   (wire (pts (xy 113.284 87.376) (xy 132.842 87.376))
+    (stroke (width 0) (type default))
+  )
+  (wire (pts (xy 104.648 98.044) (xy 104.648 97.536))
     (stroke (width 0) (type default))
   )
@@
         (path "/9c710720-cfe2-4b3b-9fda-84c630167e07/9005e841-4001-4ea2-9c18-829c9beaf08c/3dae97d6-a24d-4907-be39-d909c38c833f"
           (reference "R29") (unit 1)
+        )
+      )
+    )
+  )
+  (symbol (lib_id "power:VDD") (at 104.648 97.536 0) (unit 1)
+    (in_bom yes) (on_board yes) (dnp no) (fields_autoplaced)
+    (property "Reference" "#PWR055" (at 104.648 101.346 0)
+      (effects (font (size 1.27 1.27)) hide)
+    )
+    (property "Value" "VDD" (at 104.648 93.98 0)
+      (effects (font (size 1.27 1.27)))
+    )
+    (property "Footprint" "" (at 104.648 97.536 0)
+      (effects (font (size 1.27 1.27)) hide)
+    )
+    (property "Datasheet" "" (at 104.648 97.536 0)
+      (effects (font (size 1.27 1.27)) hide)
+    )
+    (pin "1")
+    (instances
+      (project "RoomLink"
+        (path "/9c710720-cfe2-4b3b-9fda-84c630167e07/9005e841-4001-4ea2-9c18-829c9beaf08c/3dae97d6-a24d-4907-be39-d909c38c833f"
+          (reference "#PWR055") (unit 1)
         )
       )
@@
         )
       )
-    )
-  )
-  (symbol (lib_id "power:+5V") (at 100.33 98.044 0) (unit 1)
-    (in_bom yes) (on_board yes) (dnp no) (fields_autoplaced)
-    (property "Reference" "#PWR060" (at 100.33 101.854 0)
-      (effects (font (size 1.27 1.27)) hide)
-    )
-    (property "Value" "+5V" (at 100.33 93.98 0)
-      (effects (font (size 1.27 1.27)))
-    )
-    (property "Footprint" "" (at 100.33 98.044 0)
-      (effects (font (size 1.27 1.27)) hide)
-    )
-    (property "Datasheet" "" (at 100.33 98.044 0)
-      (effects (font (size 1.27 1.27)) hide)
-    )
-    (pin "1")
-    (instances
-      (project "RoomLink"
-        (path "/9c710720-cfe2-4b3b-9fda-84c630167e07/9005e841-4001-4ea2-9c18-829c9beaf08c/3dae97d6-a24d-4907-be39-d909c38c833f"
-          (reference "#PWR060") (unit 1)
-        )
-      )
