File: Proyecto KICAD/RoomLink/INPUTS.kicad_sch (KiCad schematic)
At the start: 28 parts, among them U1 FODM214, U2 FODM214, U3 FODM214, U4 FODM214

Commit message: PCB
Connections:
- net +5V is gone; now on net VDD: R1.1, R11.1, R12.1, R15.1, R16.1, R2.1, R7.1, R8.1

Commit message: ll
Connections:
- net GND: no longer R10.2, R14.2, R4.2, R6.2
- net VDD: no longer R13.1, R3.1, R5.1, R9.1
- new net +3V3: R13.1, R3.1, R5.1, R9.1
- new net GNDA: R10.2, R14.2, R4.2, R6.2
