File: Proyecto KICAD/RoomLink/CONTROL.kicad_sch (KiCad schematic)
At the start: 11 parts, among them U10 ESP32-WROOM-32

Commit message: Room link1
Other:
- moved on the sheet: U10
Changed lines of the file:
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@@
     )
   )
-  (symbol (lib_id "RF_Module:ESP32-WROOM-32") (at 243.586 81.026 0) (unit 1)
+  (symbol (lib_id "RF_Module:ESP32-WROOM-32") (at 247.396 91.948 0) (unit 1)
     (in_bom yes) (on_board yes) (dnp no) (fields_autoplaced)
-    (property "Reference" "U10" (at 245.5419 44.45 0)
+    (property "Reference" "U10" (at 249.3519 55.372 0)
       (effects (font (size 1.27 1.27)) (justify left))
     )
-    (property "Value" "ESP32-WROOM-32" (at 245.5419 46.99 0)
+    (property "Value" "ESP32-WROOM-32" (at 249.3519 57.912 0)
       (effects (font (size 1.27 1.27)) (justify left))
     )
-    (property "Footprint" "RF_Module:ESP32-WROOM-32" (at 243.586 119.126 0)
+    (property "Footprint" "RF_Module:ESP32-WROOM-32" (at 247.396 130.048 0)
       (effects (font (size 1.27 1.27)) hide)
     )
-    (property "Datasheet" "https://www.espressif.com/sites/default/files/documentation/esp32-wroom-32_datasheet_en.pdf" (at 235.966 79.756 0)
+    (property "Datasheet" "https://www.espressif.com/sites/default/files/documentation/esp32-wroom-32_datasheet_en.pdf" (at 239.776 90.678 0)
       (effects (font (size 1.27 1.27)) hide)
     )

Commit message: PCB
Connections:
- net +5V renamed VDD

Commit message: BLLLLLL
Parts:
- removed R42: 10K, Resistor_SMD:R_0805_2012Metric, symbol Device:R
Connections:
- net COM_RS485_LCD: now also U10.6 (IO34)
- net CON_RS485_eXT: now also U10.7 (IO35)
- net GND: now also U10.1 (GND), U10.15 (GND), U10.38 (GND), U10.39 (GND)
- net INPUT_1_MICRO: now also U10.16 (IO13)
- net INPUT_2_MICRO: now also U10.14 (IO12)
- net INPUT_3_MICRO: now also U10.24 (IO2)
- net INPUT_4_MICRO: now also U10.26 (IO4)
- net RLY_FAN1_MICRO: now also U10.10 (IO25)
- net RLY_FAN2_MICRO: now also U10.11 (IO26)
- net RLY_FAN3_MICRO: now also U10.12 (IO27)
- net RLY_OUT1_MICRO: now also U10.36 (IO22)
- net RLY_OUT2_MICRO: now also U10.37 (IO23)
- net Rx_RS485_eXT: now also U10.34 (RXD0/IO3)
- net Rx_RS485_lcd: now also U10.27 (IO16)
- net Tx_RS485_LCD: now also U10.28 (IO17)
- net Tx_RS485_eXT: now also U10.35 (TXD0/IO1)
- net VDD: now also U10.2 (VDD)
- net at D21.1 (K): now also U10.13 (IO14)
Other:
- moved on the sheet: D21, J7, J8, R47, R48, R49, R50, R51, R52, U10

Commit message: Esquematico
Parts:
- removed J8: ~, Connector_PinHeader_2.54mm:PinHeader_2x03_P2.54mm_Vertical, symbol New_Library:HD-R6
- removed R52: 1K, Resistor_SMD:R_0805_2012Metric, symbol Device:R
- added C10, C12: 0.1uF, Capacitor_SMD:C_0805_2012Metric, symbol Device:C
- added C11: 22uF, Capacitor_SMD:C_0805_2012Metric, symbol Device:C
- added R34, R35: 100K, Resistor_SMD:R_0805_2012Metric, symbol Device:R
- added R36: 22K, Resistor_SMD:R_0805_2012Metric, symbol Device:R
- added U6: ~, Connector_PinHeader_2.54mm:PinHeader_2x05_P2.54mm_Vertical, symbol New_Library:ESP32-JTAG
Connections:
- net GND: now also C11.2, C12.2, U6.3 (GND), U6.9 (GND)
- net INPUT_1_MICRO: now also U10.25 (IO0); no longer U10.16 (IO13)
- net INPUT_2_MICRO: now also U10.29 (IO5); no longer U10.14 (IO12)
- net INPUT_3_MICRO: now also U10.26 (IO4); no longer U10.24 (IO2)
- net INPUT_4_MICRO: now also U10.24 (IO2); no longer U10.26 (IO4)
- net VDD: now also C10.1, C11.1, C12.1, R34.1, R35.1, R36.1
- net MTMS: now reaches R48.2
- net MTMS: now also U10.13 (IO14), U6.2 (MTMS)
- net at J7.2: now also U10.30 (IO18)
- net at J7.3: now also U10.8 (IO32)
- net at J7.4: now also U10.31 (IO19)
- net at J7.6: now also U10.33 (IO21)
- net at D21.1 (K): now also U10.9 (IO33); no longer U10.13 (IO14)
- net MTD0: now reaches U10.23 (IO15)
- net MTD0: now also R50.2, U6.6 (MTD0)
- net EN: now reaches U10.3 (EN)
- net EN: now also C10.2, R35.2, R36.2, U6.10 (EN)
- net MTCLK: now reaches R49.2
- net MTCLK: now also U10.16 (IO13), U6.4 (MTCLK)
- net at R51.2: now also U6.1 (Vin)
- new net MTD1: R34.2, U10.14 (IO12), U6.8 (MTD1)
Other:
- moved on the sheet: D21, J7, R47, R48, R49, R50, R51, U10

Commit message: ll
Other:
- moved on the sheet: R34, R35, R48, R49, R50
