File: Proyecto KICAD/RoomLink/POWER_SUPPLY.kicad_sch (KiCad schematic)
At the start: 23 parts, among them U5 LM7805_TO220, U6 B0505S-W2R2

Commit message: PCB
Parts:
- removed U5: LM7805_TO220, Package_TO_SOT_THT:TO-220-3_Vertical, symbol Regulator_Linear:LM7805_TO220
- removed U6: B0505S-W2R2, Huellas:B0505S-W2R2, symbol New_Library:B0505S-W2R2
- added PS2: B0503S-1WR3, CONV_B0503S-1WR3, symbol B0503S-1WR3:B0503S-1WR3
- added U5: ~, 3.3:DPAK228P968X238-4N, symbol New_Library:NJM2885DL1-33-TE1
- C5: value 0.1uF/25V -> 0.33uF/25V
- C6: value 0.1uF/25V -> 2.2uF/25V
Connections:
- net +5V is gone; now on net VDD: C6.1, C7.1, D5.1 (A), R20.1, TP1.1
- net +12V: now also U5.1 (VI)
- net GND: now also PS2.1 (GND), U5.2 (GND)
- net GNDREF: now also PS2.3 (0V)
- net VDD: now also PS2.2 (VIN), PS2.4 (+VO), U5.3 (VO)

Commit message: ll
Parts:
- removed D9: LED, Diode_SMD:D_0805_2012Metric, symbol Device:LED
- removed PS2: B0503S-1WR3, CONV_B0503S-1WR3, symbol B0503S-1WR3:B0503S-1WR3
- removed R19: 2.2K, Diode_SMD:D_0805_2012Metric, symbol Device:R
- added U11: B0303S, Huellas:B0505S-W2R2, symbol New_Library:B0505S-W2R2
- U5: value ~ -> NJM2885DL1-33-TE1
Connections:
- net GND: now also U11.1 (IN-)
- net VDD: now also U11.2 (IN+); no longer D6.1 (A)
- new net +3V3: D6.1 (A), U11.4 (OUT+)
- new net GNDA: U11.3 (OUT-)

Commit message: hhh
Parts:
- TP1, TP2, TP3: footprint TestPoint:TestPoint_Loop_D2.60mm_Drill1.6mm_Beaded -> TestPoint:TestPoint_Loop_D1.80mm_Drill1.0mm_Beaded
Changed lines of the file:
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@@
       (effects (font (size 1.27 1.27)) (justify left))
     )
-    (property "Footprint" "TestPoint:TestPoint_Loop_D2.60mm_Drill1.6mm_Beaded" (at 130.81 54.61 0)
+    (property "Footprint" "TestPoint:TestPoint_Loop_D1.80mm_Drill1.0mm_Beaded" (at 130.81 54.61 0)
       (effects (font (size 1.27 1.27)) hide)
     )
@@
       (effects (font (size 1.27 1.27)) (justify left))
     )
-    (property "Footprint" "TestPoint:TestPoint_Loop_D2.60mm_Drill1.6mm_Beaded" (at 88.9 55.88 0)
+    (property "Footprint" "TestPoint:TestPoint_Loop_D1.80mm_Drill1.0mm_Beaded" (at 88.9 55.88 0)
       (effects (font (size 1.27 1.27)) hide)
     )
@@
       (effects (font (size 1.27 1.27)) (justify left))
     )
-    (property "Footprint" "TestPoint:TestPoint_Loop_D2.60mm_Drill1.6mm_Beaded" (at 104.14 146.05 0)
-      (effects (font (size 1.27 1.27)) hide)
-    )
+    (property "Footprint" "TestPoint:TestPoint_Loop_D1.80mm_Drill1.0mm_Beaded" (at 104.14 146.05 0)
+      (effects (font (size 1.27 1.27)) hide)
+    )

Commit message: Raymundo
Changed lines of the file:
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@@
       (effects (font (size 1.27 1.27)))
     )
-    (property "Value" "NJM2885DL1-33-TE1" (at 110.49 55.626 0)
+    (property "Value" "NJM2885DL1-33-TE1" (at 109.982 55.626 0)
       (effects (font (size 1.27 1.27)))
     )
