File: Proyecto KICAD/RoomLink/RS-485-LCD.kicad_sch (KiCad schematic)
At the start: 8 parts, among them U7 SP485ECN-L

Commit message: PCB
Connections:
- net +5V renamed VDD
Changed lines of the file:
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@@
     (stroke (width 0) (type default))
   )
-  (wire (pts (xy 62.23 108.458) (xy 62.23 111.506))
+  (wire (pts (xy 62.23 101.346) (xy 62.23 111.506))
     (stroke (width 0) (type default))
   )
@@
     (stroke (width 0) (type default))
   )
-  (wire (pts (xy 117.602 77.978) (xy 117.602 75.692))
-    (stroke (width 0) (type default))
-  )
   (wire (pts (xy 62.23 119.126) (xy 62.23 123.698))
     (stroke (width 0) (type default))
@@
     (stroke (width 0) (type default))
   )
+  (wire (pts (xy 115.062 75.184) (xy 115.062 77.978))
+    (stroke (width 0) (type default))
+  )
   (wire (pts (xy 161.036 83.058) (xy 157.226 83.058))
     (stroke (width 0) (type default))
   )
-  (wire (pts (xy 121.666 77.978) (xy 117.602 77.978))
+  (wire (pts (xy 115.062 77.978) (xy 121.666 77.978))
     (stroke (width 0) (type default))
   )
@@
     (stroke (width 0) (type default))
   )
-  (wire (pts (xy 79.756 108.204) (xy 79.756 111.252))
+  (wire (pts (xy 79.756 101.854) (xy 79.756 111.252))
     (stroke (width 0) (type default))
   )
@@
   (hierarchical_label "CON-LCDA-" (shape bidirectional) (at 222.504 80.518 0) (fields_autoplaced)
     (effects (font (size 1.27 1.27)) (justify left))
+  )
+  (symbol (lib_id "power:VDD") (at 62.23 101.346 0) (unit 1)
+    (in_bom yes) (on_board yes) (dnp no) (fields_autoplaced)
+    (property "Reference" "#PWR053" (at 62.23 105.156 0)
+      (effects (font (size 1.27 1.27)) hide)
+    )
+    (property "Value" "VDD" (at 62.23 97.282 0)
+      (effects (font (size 1.27 1.27)))
+    )
+    (property "Footprint" "" (at 62.23 101.346 0)
+      (effects (font (size 1.27 1.27)) hide)
+    )
+    (property "Datasheet" "" (at 62.23 101.346 0)
+      (effects (font (size 1.27 1.27)) hide)
+    )
+    (pin "1")
+    (instances
+      (project "RoomLink"
+        (path "/9c710720-cfe2-4b3b-9fda-84c630167e07/9005e841-4001-4ea2-9c18-829c9beaf08c/3bf76bdf-4364-44b3-bde1-95fd668b856b"
+          (reference "#PWR053") (unit 1)
+        )
+      )
+    )
   )
   (symbol (lib_id "Device:R") (at 206.756 80.518 90) (unit 1)
@@
     )
   )
-  (symbol (lib_id "power:+5V") (at 79.756 108.204 0) (unit 1)
-    (in_bom yes) (on_board yes) (dnp no) (fields_autoplaced)
-    (property "Reference" "#PWR057" (at 79.756 112.014 0)
-      (effects (font (size 1.27 1.27)) hide)
-    )
-    (property "Value" "+5V" (at 79.756 104.902 0)
-      (effects (font (size 1.27 1.27)))
-    )
-    (property "Footprint" "" (at 79.756 108.204 0)
-      (effects (font (size 1.27 1.27)) hide)
-    )
-    (property "Datasheet" "" (at 79.756 108.204 0)
-      (effects (font (size 1.27 1.27)) hide)
-    )
-    (pin "1")
-    (instances
-      (project "RoomLink"
-        (path "/9c710720-cfe2-4b3b-9fda-84c630167e07/9005e841-4001-4ea2-9c18-829c9beaf08c/3bf76bdf-4364-44b3-bde1-95fd668b856b"
-          (reference "#PWR057") (unit 1)
-        )
-      )
-    )
-  )
-  (symbol (lib_id "power:+5V") (at 62.23 108.458 0) (unit 1)
-    (in_bom yes) (on_board yes) (dnp no) (fields_autoplaced)
-    (property "Reference" "#PWR055" (at 62.23 112.268 0)
-      (effects (font (size 1.27 1.27)) hide)
-    )
-    (property "Value" "+5V" (at 62.23 105.156 0)
-      (effects (font (size 1.27 1.27)))
-    )
-    (property "Footprint" "" (at 62.23 108.458 0)
-      (effects (font (size 1.27 1.27)) hide)
-    )
-    (property "Datasheet" "" (at 62.23 108.458 0)
-      (effects (font (size 1.27 1.27)) hide)
-    )
-    (pin "1")
-    (instances
-      (project "RoomLink"
-        (path "/9c710720-cfe2-4b3b-9fda-84c630167e07/9005e841-4001-4ea2-9c18-829c9beaf08c/3bf76bdf-4364-44b3-bde1-95fd668b856b"
-          (reference "#PWR055") (unit 1)
+  (symbol (lib_id "power:VDD") (at 115.062 75.184 0) (unit 1)
+    (in_bom yes) (on_board yes) (dnp no) (fields_autoplaced)
+    (property "Reference" "#PWR037" (at 115.062 78.994 0)
+      (effects (font (size 1.27 1.27)) hide)
+    )
+    (property "Value" "VDD" (at 115.062 71.12 0)
+      (effects (font (size 1.27 1.27)))
+    )
+    (property "Footprint" "" (at 115.062 75.184 0)
+      (effects (font (size 1.27 1.27)) hide)
+    )
+    (property "Datasheet" "" (at 115.062 75.184 0)
+      (effects (font (size 1.27 1.27)) hide)
+    )
+    (pin "1")
+    (instances
+      (project "RoomLink"
+        (path "/9c710720-cfe2-4b3b-9fda-84c630167e07/9005e841-4001-4ea2-9c18-829c9beaf08c/3bf76bdf-4364-44b3-bde1-95fd668b856b"
+          (reference "#PWR037") (unit 1)
+        )
+      )
+    )
+  )
+  (symbol (lib_id "power:VDD") (at 79.756 101.854 0) (unit 1)
+    (in_bom yes) (on_board yes) (dnp no) (fields_autoplaced)
+    (property "Reference" "#PWR063" (at 79.756 105.664 0)
+      (effects (font (size 1.27 1.27)) hide)
+    )
+    (property "Value" "VDD" (at 79.756 97.79 0)
+      (effects (font (size 1.27 1.27)))
+    )
+    (property "Footprint" "" (at 79.756 101.854 0)
+      (effects (font (size 1.27 1.27)) hide)
+    )
+    (property "Datasheet" "" (at 79.756 101.854 0)
+      (effects (font (size 1.27 1.27)) hide)
+    )
+    (pin "1")
+    (instances
+      (project "RoomLink"
+        (path "/9c710720-cfe2-4b3b-9fda-84c630167e07/9005e841-4001-4ea2-9c18-829c9beaf08c/3bf76bdf-4364-44b3-bde1-95fd668b856b"
+          (reference "#PWR063") (unit 1)
         )
       )
@@
         )
       )
-    )
-  )
-  (symbol (lib_id "power:+5V") (at 117.602 75.692 0) (unit 1)
-    (in_bom yes) (on_board yes) (dnp no) (fields_autoplaced)
-    (property "Reference" "#PWR053" (at 117.602 79.502 0)
-      (effects (font (size 1.27 1.27)) hide)
-    )
-    (property "Value" "+5V" (at 117.602 72.39 0)
-      (effects (font (size 1.27 1.27)))
-    )
-    (property "Footprint" "" (at 117.602 75.692 0)
-      (effects (font (size 1.27 1.27)) hide)
-    )
-    (property "Datasheet" "" (at 117.602 75.692 0)
-      (effects (font (size 1.27 1.27)) hide)
-    )
-    (pin "1")
-    (instances
-      (project "RoomLink"
-        (path "/9c710720-cfe2-4b3b-9fda-84c630167e07/9005e841-4001-4ea2-9c18-829c9beaf08c/3bf76bdf-4364-44b3-bde1-95fd668b856b"
-          (reference "#PWR053") (unit 1)
-        )
-      )

Commit message: Raymundo
Parts:
- U7: footprint SOIC127P600X175-8N -> SP485ECN-L:SOIC127P600X175-8N
Connections:
- net at D16.2, R28.1, U7.7 (B): now also D17.1
- net at D16.1, D17.2, R27.1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: no longer D17.1
Changed lines of the file:
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@@
   (junction (at 173.482 77.978) (diameter 0) (color 0 0 0 0)
   )
+  (junction (at 118.11 88.138) (diameter 0) (color 0 0 0 0)
+  )
+  (junction (at 177.292 80.518) (diameter 0) (color 0 0 0 0)
+  )
   (junction (at 179.832 77.978) (diameter 0) (color 0 0 0 0)
   )
-  (junction (at 118.11 88.138) (diameter 0) (color 0 0 0 0)
-  )
-  (junction (at 177.292 77.978) (diameter 0) (color 0 0 0 0)
-  )
-  (wire (pts (xy 177.292 77.978) (xy 177.292 85.344))
+  (wire (pts (xy 173.482 77.978) (xy 179.832 77.978))
+    (stroke (width 0) (type default))
+  )
+  (wire (pts (xy 183.896 73.66) (xy 183.896 80.518))
+    (stroke (width 0) (type default))
+  )
+  (wire (pts (xy 62.23 101.346) (xy 62.23 111.506))
     (stroke (width 0) (type default))
   )
@@
     (stroke (width 0) (type default))
   )
-  (wire (pts (xy 183.896 73.66) (xy 183.896 80.518))
-    (stroke (width 0) (type default))
-  )
-  (wire (pts (xy 62.23 101.346) (xy 62.23 111.506))
-    (stroke (width 0) (type default))
-  )
   (wire (pts (xy 79.756 118.872) (xy 79.756 123.444))
     (stroke (width 0) (type default))
@@
     (stroke (width 0) (type default))
   )
+  (wire (pts (xy 121.666 85.598) (xy 118.11 85.598))
+    (stroke (width 0) (type default))
+  )
+  (wire (pts (xy 62.23 119.126) (xy 62.23 123.698))
+    (stroke (width 0) (type default))
+  )
+  (wire (pts (xy 161.036 86.868) (xy 161.036 83.058))
+    (stroke (width 0) (type default))
+  )
+  (wire (pts (xy 173.482 73.66) (xy 173.482 77.978))
+    (stroke (width 0) (type default))
+  )
+  (wire (pts (xy 157.226 80.518) (xy 177.292 80.518))
+    (stroke (width 0) (type default))
+  )
+  (wire (pts (xy 109.728 88.138) (xy 118.11 88.138))
+    (stroke (width 0) (type default))
+  )
+  (wire (pts (xy 222.504 80.518) (xy 210.566 80.518))
+    (stroke (width 0) (type default))
+  )
+  (wire (pts (xy 183.642 73.66) (xy 183.896 73.66))
+    (stroke (width 0) (type default))
+  )
+  (wire (pts (xy 115.062 75.184) (xy 115.062 77.978))
+    (stroke (width 0) (type default))
+  )
+  (wire (pts (xy 161.036 83.058) (xy 157.226 83.058))
+    (stroke (width 0) (type default))
+  )
+  (wire (pts (xy 115.062 77.978) (xy 121.666 77.978))
+    (stroke (width 0) (type default))
+  )
   (wire (pts (xy 179.832 77.978) (xy 179.832 85.344))
     (stroke (width 0) (type default))
   )
-  (wire (pts (xy 121.666 85.598) (xy 118.11 85.598))
-    (stroke (width 0) (type default))
-  )
-  (wire (pts (xy 173.482 77.978) (xy 177.292 77.978))
-    (stroke (width 0) (type default))
-  )
-  (wire (pts (xy 62.23 119.126) (xy 62.23 123.698))
-    (stroke (width 0) (type default))
-  )
-  (wire (pts (xy 161.036 86.868) (xy 161.036 83.058))
-    (stroke (width 0) (type default))
-  )
-  (wire (pts (xy 173.482 73.66) (xy 173.482 77.978))
-    (stroke (width 0) (type default))
-  )
-  (wire (pts (xy 109.728 88.138) (xy 118.11 88.138))
-    (stroke (width 0) (type default))
-  )
-  (wire (pts (xy 177.292 77.978) (xy 179.832 77.978))
-    (stroke (width 0) (type default))
-  )
-  (wire (pts (xy 222.504 80.518) (xy 210.566 80.518))
-    (stroke (width 0) (type default))
-  )
-  (wire (pts (xy 183.642 73.66) (xy 183.896 73.66))
-    (stroke (width 0) (type default))
-  )
-  (wire (pts (xy 115.062 75.184) (xy 115.062 77.978))
-    (stroke (width 0) (type default))
-  )
-  (wire (pts (xy 161.036 83.058) (xy 157.226 83.058))
-    (stroke (width 0) (type default))
-  )
-  (wire (pts (xy 115.062 77.978) (xy 121.666 77.978))
-    (stroke (width 0) (type default))
-  )
   (wire (pts (xy 177.292 105.664) (xy 177.292 107.188))
     (stroke (width 0) (type default))
@@
     (stroke (width 0) (type default))
   )
+  (wire (pts (xy 177.292 80.518) (xy 183.896 80.518))
+    (stroke (width 0) (type default))
+  )
   (wire (pts (xy 79.756 101.854) (xy 79.756 111.252))
     (stroke (width 0) (type default))
@@
     (stroke (width 0) (type default))
   )
+  (wire (pts (xy 177.292 80.518) (xy 177.292 85.344))
+    (stroke (width 0) (type default))
+  )
   (wire (pts (xy 118.11 85.598) (xy 118.11 88.138))
     (stroke (width 0) (type default))
   )
   (wire (pts (xy 121.666 83.058) (xy 111.506 83.058))
-    (stroke (width 0) (type default))
-  )
-  (wire (pts (xy 157.226 80.518) (xy 183.896 80.518))
     (stroke (width 0) (type default))
   )
@@
       (effects (font (size 1.27 1.27)))
     )
-    (property "Footprint" "SOIC127P600X175-8N" (at 121.666 77.978 0)
-      (effects (font (size 1.27 1.27)) (justify bottom) hide)
-    )
+    (property "Footprint" "SP485ECN-L:SOIC127P600X175-8N" (at 121.666 77.978 0)
+      (effects (font (size 1.27 1.27)) (justify bottom) hide)
+    )
