File: Proyecto KICAD/RoomLink/RoomLink.kicad_pcb (KiCad board)
At the start: 2 copper layers, 102.4 x 83.1 mm, 103 parts, among them J1 TBP04R12-500-02BE, J2 TBP04R12-500-02BE, J3 TBP04R12-500-02BE, J4 TBP04R12-500-03GR, J5 TBP04R12-500-08GR, J6 TBP04R12-500-08GR, U1 FODM214, U10 ESP32-WROOM-32, U2 FODM214, U3 FODM214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

Commit message: Room link1
Parts:
- moved U10 0.65 mm to (181.5, 105.2)

Commit message: PCB
Parts:
- removed U6: B0505S-W2R2, Huellas:B0505S-W2R2
- added PS2: B0503S-1WR3, B0503S-1WR3:CONV_B0503S-1WR3, F.Cu at (192.8, 137.7)
- C5: value 0.1uF/25V -> 0.33uF/25V
- C6: value 0.1uF/25V -> 2.2uF/25V
- U5: value LM7805_TO220 -> ~; footprint Package_TO_SOT_THT:TO-220-3_Vertical -> 3.3:DPAK228P968X238-4N
- moved U5 18.6 mm to (24.8, 106.2)
- moved D16 1.02 mm to (184.4, 137.4)
Connections:
- C6 pad 1: +5V -> VDD
- C7 pad 1: +5V -> VDD
- C8 pad 1: +5V -> VDD
- C9 pad 1: +5V -> VDD
- D5 pad 1: +5V -> VDD
- J7 pad 1: +5V -> VDD
- R1 pad 1: +5V -> VDD
- R11 pad 1: +5V -> VDD
- R12 pad 1: +5V -> VDD
- R15 pad 1: +5V -> VDD
- R16 pad 1: +5V -> VDD
- R2 pad 1: +5V -> VDD
- R20 pad 1: +5V -> VDD
- R42 pad 1: +5V -> VDD
- R47 pad 2: +5V -> VDD
- R48 pad 1: +5V -> VDD
- R49 pad 1: +5V -> VDD
- R50 pad 1: +5V -> VDD
- R51 pad 1: +5V -> VDD
- R52 pad 1: +5V -> VDD
- R7 pad 1: +5V -> VDD
- R8 pad 1: +5V -> VDD
- TP1 pad 1: +5V -> VDD
- U5 pad 2: unconnected-(U5-GND-Pad2) -> GND
- U5 pad 3: +5V -> VDD
- U7 pad 8: +5V -> VDD
- U8 pad 1: +5V -> VDD

Commit message: Esquematico
Connections:
- D21 pad 1: unconnected-(D21-K-Pad1) -> Net-(D21-K)
- J7 pad 2: unconnected-(J7-Pad2) -> Net-(U10-IO18)
- J7 pad 3: unconnected-(J7-Pad3) -> Net-(U10-IO15)
- J7 pad 4: unconnected-(J7-Pad4) -> Net-(U10-IO19)
- J7 pad 6: unconnected-(J7-Pad6) -> Net-(U10-IO21)
- U10 pad 1: Net-(U10-GND-Pad1) -> GND
- U10 pad 10: unconnected-(U10-IO25-Pad10) -> /Smart-Control-HVAC/CONTROL/RLY_FAN1_MICRO
- U10 pad 11: unconnected-(U10-IO26-Pad11) -> /Smart-Control-HVAC/CONTROL/RLY_FAN2_MICRO
- U10 pad 12: unconnected-(U10-IO27-Pad12) -> /Smart-Control-HVAC/CONTROL/RLY_FAN3_MICRO
- U10 pad 13: unconnected-(U10-IO14-Pad13) -> Net-(D21-K)
- U10 pad 14: unconnected-(U10-IO12-Pad14) -> /Smart-Control-HVAC/CONTROL/INPUT_2_MICRO
- U10 pad 15: Net-(U10-GND-Pad1) -> GND
- U10 pad 16: unconnected-(U10-IO13-Pad16) -> /Smart-Control-HVAC/CONTROL/INPUT_1_MICRO
- U10 pad 2: unconnected-(U10-VDD-Pad2) -> VDD
- U10 pad 20: unconnected-(U10-SCK/CLK-Pad20) -> Net-(J8-SWD_CLK)
- U10 pad 21: unconnected-(U10-SDO/SD0-Pad21) -> Net-(J8-SWD_DIO)
- U10 pad 23: unconnected-(U10-IO15-Pad23) -> Net-(U10-IO15)
- U10 pad 24: unconnected-(U10-IO2-Pad24) -> /Smart-Control-HVAC/CONTROL/INPUT_3_MICRO
- U10 pad 26: unconnected-(U10-IO4-Pad26) -> /Smart-Control-HVAC/CONTROL/INPUT_4_MICRO
- U10 pad 27: unconnected-(U10-IO16-Pad27) -> /Smart-Control-HVAC/CONTROL/Rx_RS485_lcd
- U10 pad 28: unconnected-(U10-IO17-Pad28) -> /Smart-Control-HVAC/CONTROL/Tx_RS485_LCD
- U10 pad 3: unconnected-(U10-EN-Pad3) -> Net-(J8-/RESET)
- U10 pad 30: unconnected-(U10-IO18-Pad30) -> Net-(U10-IO18)
- U10 pad 31: unconnected-(U10-IO19-Pad31) -> Net-(U10-IO19)
- U10 pad 33: unconnected-(U10-IO21-Pad33) -> Net-(U10-IO21)
- U10 pad 34: unconnected-(U10-RXD0/IO3-Pad34) -> /Smart-Control-HVAC/CONTROL/Rx_RS485_eXT
- U10 pad 35: unconnected-(U10-TXD0/IO1-Pad35) -> /Smart-Control-HVAC/CONTROL/Tx_RS485_eXT
- U10 pad 36: unconnected-(U10-IO22-Pad36) -> /Smart-Control-HVAC/CONTROL/RLY_OUT1_MICRO
- U10 pad 37: unconnected-(U10-IO23-Pad37) -> /Smart-Control-HVAC/CONTROL/RLY_OUT2_MICRO
- U10 pad 38: Net-(U10-GND-Pad1) -> GND
- U10 pad 39: Net-(U10-GND-Pad1) -> GND
- U10 pad 6: unconnected-(U10-IO34-Pad6) -> /Smart-Control-HVAC/CONTROL/COM_RS485_LCD
- U10 pad 7: unconnected-(U10-IO35-Pad7) -> /Smart-Control-HVAC/CONTROL/CON_RS485_eXT

Commit message: ll
Parts:
- removed D9: LED, Diode_SMD:D_0805_2012Metric
- removed J8: ~, Connector_PinHeader_2.54mm:PinHeader_2x03_P2.54mm_Vertical
- removed PS2: B0503S-1WR3, B0503S-1WR3:CONV_B0503S-1WR3
- removed R19: 2.2K, Diode_SMD:D_0805_2012Metric
- removed R42: 10K, Resistor_SMD:R_0805_2012Metric
- removed R52: 1K, Resistor_SMD:R_0805_2012Metric
- added C10: 0.1uF, Capacitor_SMD:C_0805_2012Metric, F.Cu at (123.8, 21.6)
- added C11: 22uF, Capacitor_SMD:C_0805_2012Metric, F.Cu at (123.8, 24.6)
- added C12: 0.1uF, Capacitor_SMD:C_0805_2012Metric, F.Cu at (123.8, 27.6)
- added R34: 100K, Resistor_SMD:R_0805_2012Metric, F.Cu at (128.2, 21.5)
- added R35: 100K, Resistor_SMD:R_0805_2012Metric, F.Cu at (128.2, 24.5)
- added R36: 22K, Resistor_SMD:R_0805_2012Metric, F.Cu at (128.2, 27.4)
- added U11: B0303S, Huellas:B0505S-W2R2, F.Cu at (176.4, 144.7)
- added U6: ~, Connector_PinHeader_2.54mm:PinHeader_2x05_P2.54mm_Vertical, F.Cu at (116.7, 22.4)
- moved K1 0.22 mm to (158.5, 83.1)
Connections:
- D6 pad 1: VDD -> +3V3
- J7 pad 3: Net-(U10-IO15) -> Net-(U10-IO32)
- R10 pad 2: GND -> GNDA
- R13 pad 1: VDD -> +3V3
- R14 pad 2: GND -> GNDA
- R3 pad 1: VDD -> +3V3
- R4 pad 2: GND -> GNDA
- R48 pad 2: Net-(J8-SWD_DIO) -> MTMS
- R49 pad 2: Net-(J8-SWD_CLK) -> MTCLK
- R5 pad 1: VDD -> +3V3
- R50 pad 2: Net-(J8-/RESET) -> MTD0
- R6 pad 2: GND -> GNDA
- R9 pad 1: VDD -> +3V3
- U10 pad 13: Net-(D21-K) -> MTMS
- U10 pad 14: /Smart-Control-HVAC/CONTROL/INPUT_2_MICRO -> MTD1
- U10 pad 16: /Smart-Control-HVAC/CONTROL/INPUT_1_MICRO -> MTCLK
- U10 pad 20: Net-(J8-SWD_CLK) -> unconnected-(U10-SCK/CLK-Pad20)
- U10 pad 21: Net-(J8-SWD_DIO) -> unconnected-(U10-SDO/SD0-Pad21)
- U10 pad 23: Net-(U10-IO15) -> MTD0
- U10 pad 24: /Smart-Control-HVAC/CONTROL/INPUT_3_MICRO -> /Smart-Control-HVAC/CONTROL/INPUT_4_MICRO
- U10 pad 25: unconnected-(U10-IO0-Pad25) -> /Smart-Control-HVAC/CONTROL/INPUT_1_MICRO
- U10 pad 26: /Smart-Control-HVAC/CONTROL/INPUT_4_MICRO -> /Smart-Control-HVAC/CONTROL/INPUT_3_MICRO
- U10 pad 29: unconnected-(U10-IO5-Pad29) -> /Smart-Control-HVAC/CONTROL/INPUT_2_MICRO
- U10 pad 3: Net-(J8-/RESET) -> EN
- U10 pad 8: unconnected-(U10-IO32-Pad8) -> Net-(U10-IO32)
- U10 pad 9: unconnected-(U10-IO33-Pad9) -> Net-(D21-K)

Commit message: hhh
Parts:
- TP1, TP2, TP3: footprint TestPoint:TestPoint_Loop_D2.60mm_Drill1.6mm_Beaded -> TestPoint:TestPoint_Loop_D1.80mm_Drill1.0mm_Beaded
- U5: value ~ -> NJM2885DL1-33-TE1
- moved U5 197.0 mm to (218.4, 142.2)
- moved D6 177.3 mm to (195.6, 132.1), turned to 180 degrees
- moved U6 144.9 mm to (31.7, 139.7)
- moved R2 121.9 mm to (186.7, 129.5)
- moved R4 116.6 mm to (179.1, 138.4), turned to 90 degrees
- moved R1 116.6 mm to (179.1, 129.5)
- moved R3 116.2 mm to (179.1, 134.6), turned to -90 degrees
- moved U1 114.9 mm to (182.9, 135.9), turned to 90 degrees
- moved D1 110.5 mm to (186.7, 132.1)
- moved C1 102.0 mm to (182.9, 129.5)
- moved D16 76.9 mm to (134.6, 78.7), turned to 180 degrees
- moved J7 76.8 mm to (139.7, 40.6)
- moved K2 25.3 mm to (190.0, 81.9)
- moved K1 25.3 mm to (183.8, 81.9)
- moved F3 18.0 mm to (100.5, 133.3), turned to 0 degrees
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Other:
- copper layers 2 -> 4

Commit message: Raymundo
Parts:
- moved J7 68.4 mm to (157.5, 106.7)
- moved K1 24.3 mm to (159.5, 83.3)
- moved K2 24.1 mm to (165.9, 83.3)
- moved R4 17.7 mm to (172.7, 121.9)
- moved R3 16.9 mm to (175.6, 118.1)
- moved D17 16.4 mm to (45.7, 72.4)
- moved D1 13.2 mm to (183.2, 119.4)
- moved D2 12.3 mm to (74.9, 84.8)
- moved R7 12.0 mm to (74.2, 87.6), turned to 90 degrees
- moved U2 11.5 mm to (68.6, 87.6)
- moved U3 10.5 mm to (70.6, 98.0)
- moved U4 10.5 mm to (70.6, 102.1)
- moved R8 8.33 mm to (76.4, 87.7), turned to 90 degrees
- moved K3 8.04 mm to (172.3, 83.3)
- moved K4 7.96 mm to (178.7, 83.3)
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Connections:
- D17 pad 1: Net-(U7-A) -> Net-(U7-B)
